Commit message: steering angle 30 deg, reduce oscillation

File: autorally_description/urdf/autoRallyPlatform.urdf.xacro (robot description, xacro)
@@ -24,4 +24,5 @@
   <!-- Degree-to-radian conversions -->
   <xacro:property name="degrees_45" value="0.785398163"/>
+  <xacro:property name="degrees_30" value="0.523599"/>
   <xacro:property name="degrees_21" value="0.3665191429"/>
   <xacro:property name="degrees_90" value="1.57079633"/>
@@ -268,5 +269,5 @@
       <!-- cant the front wheels to improve traction -->
       <axis xyz="0 ${-lr_reflect*0.09950372}  0.99503719"/>
-      <limit lower="${-degrees_21}" upper="${degrees_21}"
+      <limit lower="${-degrees_30}" upper="${degrees_30}"
              effort="${servo_stall_torque}" velocity="${servo_no_load_speed}"/>
     </joint>

Commit message: disable front brake, make wheels wider, add no gui option

File: autorally_description/urdf/autoRallyPlatform.urdf.xacro (robot description, xacro)
@@ -53,5 +53,5 @@
        vertical wheel travel. -->
   <xacro:property name="wheelbase" value="0.570"/>
-  <xacro:property name="hex_hub_dist" value="0.4"/>
+  <xacro:property name="hex_hub_dist" value="0.5"/>
   <!-- <xacro:property name="axle_length" value="0.03"/> -->
   <!--<xacro:property name="wheel_travel" value="0.1"/>

Commit message: move start back, reduce ground plane friction

File: autorally_description/urdf/autoRallyPlatform.urdf.xacro (robot description, xacro)
@@ -226,26 +226,7 @@
         </geometry>
       </collision>
-      <collision name="material">
-        <origin xyz="0 0 0"/>
-        <geometry>
-          <mesh filename="${wheel_model}" />
-        </geometry>
-      </collision>
       <xacro:thick_walled_tube_inertial
           inner_rad="${hub_dia / 2.0}" outer_rad="${tire_dia / 2.0}"
           height="${tire_width}" mass="${wheel_mass}"/>
-      <max_contacts>1</max_contacts>
-      <surface>
-        <contact>
-          <ode>
-            <soft_cfm>0.000000001</soft_cfm>
-            <soft_erp>0.2</soft_erp>
-            <kp>1e+10</kp>
-            <kd>10</kd>
-            <max_vel>0.01</max_vel>
-            <min_depth>0.005</min_depth>
-          </ode>
-        </contact>
-      </surface>
     </link>
     <gazebo reference="${lr_prefix}_${fr_prefix}_wheel">

Commit message: friction to 0.9 and wheel width to 0.4 to allow rolling over

File: autorally_description/urdf/autoRallyPlatform.urdf.xacro (robot description, xacro)
@@ -53,5 +53,6 @@
        vertical wheel travel. -->
   <xacro:property name="wheelbase" value="0.570"/>
-  <xacro:property name="hex_hub_dist" value="0.5"/>
+  <!-- <xacro:property name="hex_hub_dist" value="0.5"/> -->
+  <xacro:property name="hex_hub_dist" value="0.4"/>
   <!-- <xacro:property name="axle_length" value="0.03"/> -->
   <!--<xacro:property name="wheel_travel" value="0.1"/>

Commit message: Adjust friction, set steering input to radians

File: autorally_description/urdf/autoRallyPlatform.urdf.xacro (robot description, xacro)
@@ -53,6 +53,6 @@
        vertical wheel travel. -->
   <xacro:property name="wheelbase" value="0.570"/>
-  <!-- <xacro:property name="hex_hub_dist" value="0.5"/> -->
-  <xacro:property name="hex_hub_dist" value="0.4"/>
+  <!-- <xacro:property name="hex_hub_dist" value="0.6"/> -->
+  <xacro:property name="hex_hub_dist" value="0.45"/>
   <!-- <xacro:property name="axle_length" value="0.03"/> -->
   <!--<xacro:property name="wheel_travel" value="0.1"/>

Commit message: wide wheels

File: autorally_description/urdf/autoRallyPlatform.urdf.xacro (robot description, xacro)
@@ -53,6 +53,6 @@
        vertical wheel travel. -->
   <xacro:property name="wheelbase" value="0.570"/>
-  <!-- <xacro:property name="hex_hub_dist" value="0.6"/> -->
-  <xacro:property name="hex_hub_dist" value="0.45"/>
+  <xacro:property name="hex_hub_dist" value="0.6"/>
+  <!-- <xacro:property name="hex_hub_dist" value="0.45"/> -->
   <!-- <xacro:property name="axle_length" value="0.03"/> -->
   <!--<xacro:property name="wheel_travel" value="0.1"/>
